Commit message: support ros kinetec 32bit and melodic

File: dsr_description/xacro/m0609.urdf.xacro (robot description, xacro)
@@ -2,5 +2,7 @@
 <robot xmlns:xacro="http://ros.org/wiki/xacro" name="m0609" >
   <xacro:arg name="color"   default="white"/>
+  <xacro:arg name="gripper" default="none"/>
   <xacro:property name="cr" value="$(arg color)"/>
+  <xacro:property name="gr" value="$(arg gripper)"/>
   <xacro:if value="${cr == 'white'}">
      <xacro:include filename="$(find dsr_description)/xacro/macro.m0609.white.xacro" />
@@ -8,4 +10,7 @@
   <xacro:if value="${cr == 'blue'}">
      <xacro:include filename="$(find dsr_description)/xacro/macro.m0609.blue.xacro" />
+  </xacro:if>
+  <xacro:if value="${gr == 'robotiq_2f'}">
+     <xacro:include filename="$(find dsr_description)/xacro/robotiq_2f.urdf.xacro" />
   </xacro:if>
   <xacro:m0609 namespace="$(arg namespace)"/>

File: dsr_description/xacro/m0617.urdf.xacro (robot description, xacro)
@@ -2,5 +2,7 @@
 <robot xmlns:xacro="http://ros.org/wiki/xacro" name="m0617" >
   <xacro:arg name="color"   default="white"/>
+  <xacro:arg name="gripper" default="robotiq_2f"/>
   <xacro:property name="cr" value="$(arg color)"/>
+  <xacro:property name="gr" value="$(arg gripper)"/>
   <xacro:if value="${cr == 'white'}">
      <xacro:include filename="$(find dsr_description)/xacro/macro.m0617.white.xacro" />
@@ -10,4 +12,7 @@
   </xacro:if>
   <xacro:m0617 namespace="$(arg namespace)"/>
+  <xacro:if value="${gr == 'robotiq_2f'}">
+     <xacro:include filename="$(find dsr_description)/xacro/robotiq_2f.urdf.xacro" />
+  </xacro:if>
   <link name="world" />
   <!-- World fixed joint-->

File: dsr_description/xacro/m1509.urdf.xacro (robot description, xacro)
@@ -2,5 +2,7 @@
 <robot xmlns:xacro="http://ros.org/wiki/xacro" name="m1509" >
   <xacro:arg name="color"   default="white"/>
+  <xacro:arg name="gripper" default="none"/>
   <xacro:property name="cr" value="$(arg color)"/>
+  <xacro:property name="gr" value="$(arg gripper)"/>
   <xacro:if value="${cr == 'white'}">
      <xacro:include filename="$(find dsr_description)/xacro/macro.m1509.white.xacro" />
@@ -8,4 +10,7 @@
   <xacro:if value="${cr == 'blue'}">
      <xacro:include filename="$(find dsr_description)/xacro/macro.m1509.blue.xacro" />
+  </xacro:if>
+  <xacro:if value="${gr == 'robotiq_2f'}">
+     <xacro:include filename="$(find dsr_description)/xacro/robotiq_2f.urdf.xacro" />
   </xacro:if>
   <xacro:m1509 namespace="$(arg namespace)"/>
