Commit message: update joint angle in URDF

File: dsr_description/xacro/macro.a0509.blue.xacro (robot description, xacro)
@@ -59,5 +59,5 @@
 			<origin rpy="0 -1.571 -1.571" xyz="0 0 0" />
 			<axis xyz="0 0 1" />
-			<limit effort="3460" lower="-6.283" upper="6.283" velocity="2.094" />
+			<limit effort="3460" lower="-1.658" upper="1.658" velocity="2.094" />
 			<dynamics friction="0" />
 		</joint>
@@ -93,5 +93,5 @@
 			<origin rpy="0 0 1.571" xyz="0.409 0 0" />
 			<axis xyz="0 0 1" />
-			<limit effort="1630" lower="-2.793" upper="2.793" velocity="3.142" />
+			<limit effort="1630" lower="-2.356" upper="2.356" velocity="3.142" />
 			<dynamics friction="0" />
 		</joint>
@@ -149,5 +149,5 @@
 			<origin rpy="-1.571 0 0" xyz="0 0 0" />
 			<axis xyz="0 0 1" />
-			<limit effort="50" lower="-6.283" upper="6.283" velocity="3.927" />
+			<limit effort="50" lower="-2.356" upper="2.356" velocity="3.927" />
 			<dynamics friction="0" />
 		</joint>

File: dsr_description/xacro/macro.m0609.blue.xacro (robot description, xacro)
@@ -47,5 +47,5 @@
 			<origin rpy="0 -1.571 -1.571" xyz="0 0.0062 0" />
 			<axis xyz="0 0 1" />
-			<limit effort="3460" lower="-6.283" upper="6.283" velocity="2.094" />
+			<limit effort="3460" lower="-1.65806" upper="1.65806" velocity="2.094" />
 			<dynamics friction="0" />
 		</joint>
@@ -81,5 +81,5 @@
 			<origin rpy="0 0 1.571" xyz="0.411 0 0" />
 			<axis xyz="0 0 1" />
-			<limit effort="1630" lower="-2.793" upper="2.793" velocity="3.142" />
+			<limit effort="1630" lower="-2.35619" upper="2.35619" velocity="3.142" />
 			<dynamics friction="0" />
 		</joint>
@@ -131,5 +131,5 @@
 			<origin rpy="-1.571 0 0" xyz="0 0 0" />
 			<axis xyz="0 0 1" />
-			<limit effort="50" lower="-6.283" upper="6.283" velocity="3.927" />
+			<limit effort="50" lower="-2.35619" upper="2.35619" velocity="3.927" />
 			<dynamics friction="0" />
 		</joint>

File: dsr_description/xacro/macro.m0609.white.xacro (robot description, xacro)
@@ -47,5 +47,5 @@
 			<origin rpy="0 -1.571 -1.571" xyz="0 0.0062 0" />
 			<axis xyz="0 0 1" />
-			<limit effort="3460" lower="-6.283" upper="6.283" velocity="2.094" />
+			<limit effort="3460" lower="-1.658" upper="1.658" velocity="2.094" />
 			<dynamics friction="0" />
 		</joint>
@@ -81,5 +81,5 @@
 			<origin rpy="0 0 1.571" xyz="0.411 0 0" />
 			<axis xyz="0 0 1" />
-			<limit effort="1630" lower="-2.793" upper="2.793" velocity="3.142" />
+			<limit effort="1630" lower="-2.356" upper="2.356" velocity="3.142" />
 			<dynamics friction="0" />
 		</joint>
@@ -131,5 +131,5 @@
 			<origin rpy="-1.571 0 0" xyz="0 0 0" />
 			<axis xyz="0 0 1" />
-			<limit effort="50" lower="-6.283" upper="6.283" velocity="3.927" />
+			<limit effort="50" lower="-2.356" upper="2.356" velocity="3.927" />
 			<dynamics friction="0" />
 		</joint>

File: dsr_description/xacro/macro.m0617.blue.xacro (robot description, xacro)
@@ -47,5 +47,5 @@
 			<origin rpy="0 -1.571 -1.571" xyz="0 0.0345 0" />
 			<axis xyz="0 0 1" />
-			<limit effort="3460" lower="-6.283" upper="6.283" velocity="2.094" />
+			<limit effort="3460" lower="-1.658" upper="1.658" velocity="2.094" />
 			<dynamics friction="0" />
 		</joint>
@@ -81,5 +81,5 @@
 			<origin rpy="0 0 1.571" xyz="0.845 0 0" />
 			<axis xyz="0 0 1" />
-			<limit effort="1630" lower="-2.793" upper="2.793" velocity="3.142" />
+			<limit effort="1630" lower="-2.356" upper="2.356" velocity="3.142" />
 			<dynamics friction="0" />
 		</joint>
@@ -131,5 +131,5 @@
 			<origin rpy="-1.571 0 0" xyz="0 0 0" />
 			<axis xyz="0 0 1" />
-			<limit effort="50" lower="-6.283" upper="6.283" velocity="3.927" />
+			<limit effort="50" lower="-2.356" upper="2.356" velocity="3.927" />
 			<dynamics friction="0" />
 		</joint>

File: dsr_description/xacro/macro.m0617.white.xacro (robot description, xacro)
@@ -47,5 +47,5 @@
 			<origin rpy="0 -1.571 -1.571" xyz="0 0.0345 0" />
 			<axis xyz="0 0 1" />
-			<limit effort="3460" lower="-6.283" upper="6.283" velocity="2.094" />
+			<limit effort="3460" lower="-1.658" upper="1.658" velocity="2.094" />
 			<dynamics friction="0" />
 		</joint>
@@ -81,5 +81,5 @@
 			<origin rpy="0 0 1.571" xyz="0.845 0 0" />
 			<axis xyz="0 0 1" />
-			<limit effort="1630" lower="-2.793" upper="2.793" velocity="3.142" />
+			<limit effort="1630" lower="-2.356" upper="2.365" velocity="3.142" />
 			<dynamics friction="0" />
 		</joint>
@@ -131,5 +131,5 @@
 			<origin rpy="-1.571 0 0" xyz="0 0 0" />
 			<axis xyz="0 0 1" />
-			<limit effort="50" lower="-6.283" upper="6.283" velocity="3.927" />
+			<limit effort="50" lower="-2.356" upper="2.356" velocity="3.927" />
 			<dynamics friction="0" />
 		</joint>

File: dsr_description/xacro/macro.m1013.blue.xacro (robot description, xacro)
@@ -47,5 +47,5 @@
 			<origin rpy="0 -1.571 -1.571" xyz="0 0.0345 0" />
 			<axis xyz="0 0 1" />
-			<limit effort="3460" lower="-6.283" upper="6.283" velocity="2.094" />
+			<limit effort="3460" lower="-1.658" upper="1.658" velocity="2.094" />
 			<dynamics friction="0" />
 		</joint>
@@ -81,5 +81,5 @@
 			<origin rpy="0 0 1.571" xyz="0.62 0 0" />
 			<axis xyz="0 0 1" />
-			<limit effort="1630" lower="-2.793" upper="2.793" velocity="3.142" />
+			<limit effort="1630" lower="-2.356" upper="2.356" velocity="3.142" />
 			<dynamics friction="0" />
 		</joint>
@@ -131,5 +131,5 @@
 			<origin rpy="-1.571 0 0" xyz="0 0 0" />
 			<axis xyz="0 0 1" />
-			<limit effort="50" lower="-6.283" upper="6.283" velocity="3.927" />
+			<limit effort="50" lower="-2.356" upper="2.356" velocity="3.927" />
 			<dynamics friction="0" />
 		</joint>

File: dsr_description/xacro/macro.m1013.white.xacro (robot description, xacro)
@@ -47,5 +47,5 @@
 			<origin rpy="0 -1.571 -1.571" xyz="0 0.0345 0" />
 			<axis xyz="0 0 1" />
-			<limit effort="3460" lower="-6.283" upper="6.283" velocity="2.094" />
+			<limit effort="3460" lower="-1.658" upper="1.658" velocity="2.094" />
 			<dynamics friction="0" />
 		</joint>
@@ -81,5 +81,5 @@
 			<origin rpy="0 0 1.571" xyz="0.62 0 0" />
 			<axis xyz="0 0 1" />
-			<limit effort="1630" lower="-2.793" upper="2.793" velocity="3.142" />
+			<limit effort="1630" lower="-2.356" upper="2.356" velocity="3.142" />
 			<dynamics friction="0" />
 		</joint>
@@ -131,5 +131,5 @@
 			<origin rpy="-1.571 0 0" xyz="0 0 0" />
 			<axis xyz="0 0 1" />
-			<limit effort="50" lower="-6.283" upper="6.283" velocity="3.927" />
+			<limit effort="50" lower="-2.356" upper="2.356" velocity="3.927" />
 			<dynamics friction="0" />
 		</joint>

File: dsr_description/xacro/macro.m1509.blue.xacro (robot description, xacro)
@@ -47,5 +47,5 @@
 			<origin rpy="0 -1.571 -1.571" xyz="0 0.0345 0" />
 			<axis xyz="0 0 1" />
-			<limit effort="3460" lower="-6.283" upper="6.283" velocity="2.094" />
+			<limit effort="3460" lower="-1.658" upper="1.658" velocity="2.094" />
 			<dynamics friction="0" />
 		</joint>
@@ -81,5 +81,5 @@
 			<origin rpy="0 0 1.571" xyz="0.411 0 0" />
 			<axis xyz="0 0 1" />
-			<limit effort="1630" lower="-2.793" upper="2.793" velocity="3.142" />
+			<limit effort="1630" lower="-2.356" upper="2.356" velocity="3.142" />
 			<dynamics friction="0" />
 		</joint>
@@ -131,5 +131,5 @@
 			<origin rpy="-1.571 0 0" xyz="0 0 0" />
 			<axis xyz="0 0 1" />
-			<limit effort="50" lower="-6.283" upper="6.283" velocity="3.927" />
+			<limit effort="50" lower="-2.356" upper="2.356" velocity="3.927" />
 			<dynamics friction="0" />
 		</joint>

File: dsr_description/xacro/macro.m1509.white.xacro (robot description, xacro)
@@ -47,5 +47,5 @@
 			<origin rpy="0 -1.571 -1.571" xyz="0 0.0345 0" />
 			<axis xyz="0 0 1" />
-			<limit effort="3460" lower="-6.283" upper="6.283" velocity="2.094" />
+			<limit effort="3460" lower="-1.658" upper="1.658" velocity="2.094" />
 			<dynamics friction="0" />
 		</joint>
@@ -81,5 +81,5 @@
 			<origin rpy="0 0 1.571" xyz="0.411 0 0" />
 			<axis xyz="0 0 1" />
-			<limit effort="1630" lower="-2.793" upper="2.793" velocity="3.142" />
+			<limit effort="1630" lower="-2.356" upper="2.356" velocity="3.142" />
 			<dynamics friction="0" />
 		</joint>
@@ -131,5 +131,5 @@
 			<origin rpy="-1.571 0 0" xyz="0 0 0" />
 			<axis xyz="0 0 1" />
-			<limit effort="50" lower="-6.283" upper="6.283" velocity="3.927" />
+			<limit effort="50" lower="-2.356" upper="2.356" velocity="3.927" />
 			<dynamics friction="0" />
 		</joint>
