Commit message: add a0912 model

File: dsr_description/xacro/a0912.urdf.xacro (robot description, xacro)
@@ -1,4 +1,4 @@
 <?xml version="1.0"?>
-<robot xmlns:xacro="http://www.ros.org/wiki/xacro" name="a0509" >
+<robot xmlns:xacro="http://www.ros.org/wiki/xacro" name="a0912" >
   <xacro:arg name="color"   default="white"/>
   <xacro:arg name="gripper" default="none"/>
@@ -6,10 +6,10 @@
   <xacro:property name="gr" value="$(arg gripper)"/>
   <xacro:if value="${cr == 'white'}">
-     <xacro:include filename="$(find dsr_description)/xacro/macro.a0509.white.xacro" />
+     <xacro:include filename="$(find dsr_description)/xacro/macro.a0912.white.xacro" />
   </xacro:if>
   <xacro:if value="${cr == 'blue'}">
-     <xacro:include filename="$(find dsr_description)/xacro/macro.a0509.blue.xacro" />
+     <xacro:include filename="$(find dsr_description)/xacro/macro.a0912.blue.xacro" />
   </xacro:if>
-  <xacro:a0509 namespace="$(arg namespace)"/>
+  <xacro:a0912 namespace="$(arg namespace)"/>
   <link name="world" />
   <xacro:if value="${gr == 'robotiq_2f'}">

File: dsr_description/xacro/a0912mobile.urdf.xacro (robot description, xacro)
@@ -1,4 +1,4 @@
 <?xml version="1.0"?>
-<robot xmlns:xacro="http://www.ros.org/wiki/xacro" name="a0509mobile" >
+<robot xmlns:xacro="http://www.ros.org/wiki/xacro" name="a0912mobile" >
   <xacro:arg name="color"   default="white"/>
   <xacro:arg name="gripper" default="none"/>
@@ -6,12 +6,12 @@
   <xacro:property name="gr" value="$(arg gripper)"/>
   <xacro:if value="${cr == 'white'}">
-    <xacro:include filename="$(find dsr_description)/xacro/macro.a0509mobile.white.xacro" />
+    <xacro:include filename="$(find dsr_description)/xacro/macro.a0912mobile.white.xacro" />
   </xacro:if>
   <xacro:if value="${cr == 'blue'}">
-    <xacro:include filename="$(find dsr_description)/xacro/macro.a0509mobile.blue.xacro" />
+    <xacro:include filename="$(find dsr_description)/xacro/macro.a0912mobile.blue.xacro" />
   </xacro:if>
   <xacro:if value="${gr == 'robotiq_2f'}">
      <xacro:include filename="$(find dsr_description)/xacro/robotiq_2f.urdf.xacro" />
   </xacro:if>
-  <xacro:a0509mobile namespace="$(arg namespace)"/>
+  <xacro:a0912mobile namespace="$(arg namespace)"/>
 </robot>

File: dsr_description/xacro/macro.m1013.blue.xacro (robot description, xacro)
@@ -151,5 +151,5 @@
 			<parent link="link5" />
 			<child link="link6" />
-			<origin rpy="1.571 0 0" xyz="0 -0.121 0" />
+			<origin rpy="1.571 0 0" xyz="0 -0.124 0" />
 			<axis xyz="0 0 1" />
 			<limit effort="50" lower="-6.283" upper="6.283" velocity="3.927" />
