Commit message: modify husky mobile mass

File: dsr_description/xacro/macro.a0509mobile.blue.xacro (robot description, xacro)
@@ -48,5 +48,5 @@
 		<link name="inertial_link">
 			<inertial>
-				<mass value="46.034" />
+				<mass value="1346.034" />
 				<origin xyz="-0.00065 -0.085 0.062" />
 				<inertia ixx="0.6022" ixy="-0.02364" ixz="-0.1197" iyy="1.7386" iyz="-0.001544" izz="2.0296" />

File: dsr_description/xacro/macro.a0509mobile.white.xacro (robot description, xacro)
@@ -48,5 +48,5 @@
 		<link name="inertial_link">
 			<inertial>
-				<mass value="46.034" />
+				<mass value="1346.034" />
 				<origin xyz="-0.00065 -0.085 0.062" />
 				<inertia ixx="0.6022" ixy="-0.02364" ixz="-0.1197" iyy="1.7386" iyz="-0.001544" izz="2.0296" />

File: dsr_description/xacro/macro.a0912mobile.blue.xacro (robot description, xacro)
@@ -48,5 +48,5 @@
 		<link name="inertial_link">
 			<inertial>
-				<mass value="46.034" />
+				<mass value="1346.034" />
 				<origin xyz="-0.00065 -0.085 0.062" />
 				<inertia ixx="0.6022" ixy="-0.02364" ixz="-0.1197" iyy="1.7386" iyz="-0.001544" izz="2.0296" />

File: dsr_description/xacro/macro.a0912mobile.white.xacro (robot description, xacro)
@@ -48,5 +48,5 @@
 		<link name="inertial_link">
 			<inertial>
-				<mass value="46.034" />
+				<mass value="1346.034" />
 				<origin xyz="-0.00065 -0.085 0.062" />
 				<inertia ixx="0.6022" ixy="-0.02364" ixz="-0.1197" iyy="1.7386" iyz="-0.001544" izz="2.0296" />

File: dsr_description/xacro/macro.m0609mobile.blue.xacro (robot description, xacro)
@@ -48,5 +48,5 @@
 		<link name="inertial_link">
 			<inertial>
-				<mass value="46.034" />
+				<mass value="1346.034" />
 				<origin xyz="-0.00065 -0.085 0.062" />
 				<inertia ixx="0.6022" ixy="-0.02364" ixz="-0.1197" iyy="1.7386" iyz="-0.001544" izz="2.0296" />

File: dsr_description/xacro/macro.m0609mobile.white.xacro (robot description, xacro)
@@ -48,5 +48,5 @@
 		<link name="inertial_link">
 			<inertial>
-				<mass value="46.034" />
+				<mass value="1346.034" />
 				<origin xyz="-0.00065 -0.085 0.062" />
 				<inertia ixx="0.6022" ixy="-0.02364" ixz="-0.1197" iyy="1.7386" iyz="-0.001544" izz="2.0296" />

File: dsr_description/xacro/macro.m0617mobile.blue.xacro (robot description, xacro)
@@ -48,5 +48,5 @@
 		<link name="inertial_link">
 			<inertial>
-				<mass value="46.034" />
+				<mass value="1346.034" />
 				<origin xyz="-0.00065 -0.085 0.062" />
 				<inertia ixx="0.6022" ixy="-0.02364" ixz="-0.1197" iyy="1.7386" iyz="-0.001544" izz="2.0296" />

File: dsr_description/xacro/macro.m0617mobile.white.xacro (robot description, xacro)
@@ -48,5 +48,5 @@
 		<link name="inertial_link">
 			<inertial>
-				<mass value="46.034" />
+				<mass value="1346.034" />
 				<origin xyz="-0.00065 -0.085 0.062" />
 				<inertia ixx="0.6022" ixy="-0.02364" ixz="-0.1197" iyy="1.7386" iyz="-0.001544" izz="2.0296" />

File: dsr_description/xacro/macro.m1013mobile.blue.xacro (robot description, xacro)
@@ -48,5 +48,5 @@
 		<link name="inertial_link">
 			<inertial>
-				<mass value="46.034" />
+				<mass value="1346.034" />
 				<origin xyz="-0.00065 -0.085 0.062" />
 				<inertia ixx="0.6022" ixy="-0.02364" ixz="-0.1197" iyy="1.7386" iyz="-0.001544" izz="2.0296" />

File: dsr_description/xacro/macro.m1013mobile.white.xacro (robot description, xacro)
@@ -48,5 +48,5 @@
 		<link name="inertial_link">
 			<inertial>
-				<mass value="46.034" />
+				<mass value="1346.034" />
 				<origin xyz="-0.00065 -0.085 0.062" />
 				<inertia ixx="0.6022" ixy="-0.02364" ixz="-0.1197" iyy="1.7386" iyz="-0.001544" izz="2.0296" />

File: dsr_description/xacro/macro.m1509mobile.blue.xacro (robot description, xacro)
@@ -48,5 +48,5 @@
 		<link name="inertial_link">
 			<inertial>
-				<mass value="46.034" />
+				<mass value="1346.034" />
 				<origin xyz="-0.00065 -0.085 0.062" />
 				<inertia ixx="0.6022" ixy="-0.02364" ixz="-0.1197" iyy="1.7386" iyz="-0.001544" izz="2.0296" />

File: dsr_description/xacro/macro.m1509mobile.white.xacro (robot description, xacro)
@@ -48,5 +48,5 @@
 		<link name="inertial_link">
 			<inertial>
-				<mass value="46.034" />
+				<mass value="1346.034" />
 				<origin xyz="-0.00065 -0.085 0.062" />
 				<inertia ixx="0.6022" ixy="-0.02364" ixz="-0.1197" iyy="1.7386" iyz="-0.001544" izz="2.0296" />

Commit message: modify husky mass

File: dsr_description/xacro/macro.a0509mobile.blue.xacro (robot description, xacro)
@@ -48,5 +48,5 @@
 		<link name="inertial_link">
 			<inertial>
-				<mass value="46.034" />
+				<mass value="346.034" />
 				<origin xyz="-0.00065 -0.085 0.062" />
 				<inertia ixx="0.6022" ixy="-0.02364" ixz="-0.1197" iyy="1.7386" iyz="-0.001544" izz="2.0296" />

File: dsr_description/xacro/macro.a0509mobile.white.xacro (robot description, xacro)
@@ -48,5 +48,5 @@
 		<link name="inertial_link">
 			<inertial>
-				<mass value="46.034" />
+				<mass value="346.034" />
 				<origin xyz="-0.00065 -0.085 0.062" />
 				<inertia ixx="0.6022" ixy="-0.02364" ixz="-0.1197" iyy="1.7386" iyz="-0.001544" izz="2.0296" />

File: dsr_description/xacro/macro.a0912mobile.blue.xacro (robot description, xacro)
@@ -48,5 +48,5 @@
 		<link name="inertial_link">
 			<inertial>
-				<mass value="46.034" />
+				<mass value="346.034" />
 				<origin xyz="-0.00065 -0.085 0.062" />
 				<inertia ixx="0.6022" ixy="-0.02364" ixz="-0.1197" iyy="1.7386" iyz="-0.001544" izz="2.0296" />

File: dsr_description/xacro/macro.a0912mobile.white.xacro (robot description, xacro)
@@ -48,5 +48,5 @@
 		<link name="inertial_link">
 			<inertial>
-				<mass value="46.034" />
+				<mass value="346.034" />
 				<origin xyz="-0.00065 -0.085 0.062" />
 				<inertia ixx="0.6022" ixy="-0.02364" ixz="-0.1197" iyy="1.7386" iyz="-0.001544" izz="2.0296" />

File: dsr_description/xacro/macro.m0609mobile.blue.xacro (robot description, xacro)
@@ -48,5 +48,5 @@
 		<link name="inertial_link">
 			<inertial>
-				<mass value="46.034" />
+				<mass value="346.034" />
 				<origin xyz="-0.00065 -0.085 0.062" />
 				<inertia ixx="0.6022" ixy="-0.02364" ixz="-0.1197" iyy="1.7386" iyz="-0.001544" izz="2.0296" />

File: dsr_description/xacro/macro.m0609mobile.white.xacro (robot description, xacro)
@@ -48,5 +48,5 @@
 		<link name="inertial_link">
 			<inertial>
-				<mass value="46.034" />
+				<mass value="346.034" />
 				<origin xyz="-0.00065 -0.085 0.062" />
 				<inertia ixx="0.6022" ixy="-0.02364" ixz="-0.1197" iyy="1.7386" iyz="-0.001544" izz="2.0296" />

File: dsr_description/xacro/macro.m0617mobile.blue.xacro (robot description, xacro)
@@ -48,5 +48,5 @@
 		<link name="inertial_link">
 			<inertial>
-				<mass value="46.034" />
+				<mass value="346.034" />
 				<origin xyz="-0.00065 -0.085 0.062" />
 				<inertia ixx="0.6022" ixy="-0.02364" ixz="-0.1197" iyy="1.7386" iyz="-0.001544" izz="2.0296" />

File: dsr_description/xacro/macro.m0617mobile.white.xacro (robot description, xacro)
@@ -48,5 +48,5 @@
 		<link name="inertial_link">
 			<inertial>
-				<mass value="46.034" />
+				<mass value="346.034" />
 				<origin xyz="-0.00065 -0.085 0.062" />
 				<inertia ixx="0.6022" ixy="-0.02364" ixz="-0.1197" iyy="1.7386" iyz="-0.001544" izz="2.0296" />

File: dsr_description/xacro/macro.m1013mobile.blue.xacro (robot description, xacro)
@@ -48,5 +48,5 @@
 		<link name="inertial_link">
 			<inertial>
-				<mass value="46.034" />
+				<mass value="346.034" />
 				<origin xyz="-0.00065 -0.085 0.062" />
 				<inertia ixx="0.6022" ixy="-0.02364" ixz="-0.1197" iyy="1.7386" iyz="-0.001544" izz="2.0296" />

File: dsr_description/xacro/macro.m1013mobile.white.xacro (robot description, xacro)
@@ -48,5 +48,5 @@
 		<link name="inertial_link">
 			<inertial>
-				<mass value="46.034" />
+				<mass value="346.034" />
 				<origin xyz="-0.00065 -0.085 0.062" />
 				<inertia ixx="0.6022" ixy="-0.02364" ixz="-0.1197" iyy="1.7386" iyz="-0.001544" izz="2.0296" />

File: dsr_description/xacro/macro.m1509mobile.blue.xacro (robot description, xacro)
@@ -48,5 +48,5 @@
 		<link name="inertial_link">
 			<inertial>
-				<mass value="46.034" />
+				<mass value="346.034" />
 				<origin xyz="-0.00065 -0.085 0.062" />
 				<inertia ixx="0.6022" ixy="-0.02364" ixz="-0.1197" iyy="1.7386" iyz="-0.001544" izz="2.0296" />

File: dsr_description/xacro/macro.m1509mobile.white.xacro (robot description, xacro)
@@ -48,5 +48,5 @@
 		<link name="inertial_link">
 			<inertial>
-				<mass value="46.034" />
+				<mass value="346.034" />
 				<origin xyz="-0.00065 -0.085 0.062" />
 				<inertia ixx="0.6022" ixy="-0.02364" ixz="-0.1197" iyy="1.7386" iyz="-0.001544" izz="2.0296" />

Commit message: add h-seires model

File: dsr_description/xacro/macro.a0509mobile.blue.xacro (robot description, xacro)
@@ -48,5 +48,5 @@
 		<link name="inertial_link">
 			<inertial>
-				<mass value="346.034" />
+				<mass value="1346.034" />
 				<origin xyz="-0.00065 -0.085 0.062" />
 				<inertia ixx="0.6022" ixy="-0.02364" ixz="-0.1197" iyy="1.7386" iyz="-0.001544" izz="2.0296" />

File: dsr_description/xacro/macro.a0509mobile.white.xacro (robot description, xacro)
@@ -48,5 +48,5 @@
 		<link name="inertial_link">
 			<inertial>
-				<mass value="346.034" />
+				<mass value="1346.034" />
 				<origin xyz="-0.00065 -0.085 0.062" />
 				<inertia ixx="0.6022" ixy="-0.02364" ixz="-0.1197" iyy="1.7386" iyz="-0.001544" izz="2.0296" />

File: dsr_description/xacro/macro.a0912mobile.blue.xacro (robot description, xacro)
@@ -48,5 +48,5 @@
 		<link name="inertial_link">
 			<inertial>
-				<mass value="346.034" />
+				<mass value="1346.034" />
 				<origin xyz="-0.00065 -0.085 0.062" />
 				<inertia ixx="0.6022" ixy="-0.02364" ixz="-0.1197" iyy="1.7386" iyz="-0.001544" izz="2.0296" />

File: dsr_description/xacro/macro.a0912mobile.white.xacro (robot description, xacro)
@@ -48,5 +48,5 @@
 		<link name="inertial_link">
 			<inertial>
-				<mass value="346.034" />
+				<mass value="1346.034" />
 				<origin xyz="-0.00065 -0.085 0.062" />
 				<inertia ixx="0.6022" ixy="-0.02364" ixz="-0.1197" iyy="1.7386" iyz="-0.001544" izz="2.0296" />

File: dsr_description/xacro/macro.m0609mobile.blue.xacro (robot description, xacro)
@@ -48,5 +48,5 @@
 		<link name="inertial_link">
 			<inertial>
-				<mass value="346.034" />
+				<mass value="1346.034" />
 				<origin xyz="-0.00065 -0.085 0.062" />
 				<inertia ixx="0.6022" ixy="-0.02364" ixz="-0.1197" iyy="1.7386" iyz="-0.001544" izz="2.0296" />

File: dsr_description/xacro/macro.m0609mobile.white.xacro (robot description, xacro)
@@ -48,5 +48,5 @@
 		<link name="inertial_link">
 			<inertial>
-				<mass value="346.034" />
+				<mass value="1346.034" />
 				<origin xyz="-0.00065 -0.085 0.062" />
 				<inertia ixx="0.6022" ixy="-0.02364" ixz="-0.1197" iyy="1.7386" iyz="-0.001544" izz="2.0296" />

File: dsr_description/xacro/macro.m0617mobile.blue.xacro (robot description, xacro)
@@ -48,5 +48,5 @@
 		<link name="inertial_link">
 			<inertial>
-				<mass value="346.034" />
+				<mass value="1346.034" />
 				<origin xyz="-0.00065 -0.085 0.062" />
 				<inertia ixx="0.6022" ixy="-0.02364" ixz="-0.1197" iyy="1.7386" iyz="-0.001544" izz="2.0296" />

File: dsr_description/xacro/macro.m0617mobile.white.xacro (robot description, xacro)
@@ -48,5 +48,5 @@
 		<link name="inertial_link">
 			<inertial>
-				<mass value="346.034" />
+				<mass value="1346.034" />
 				<origin xyz="-0.00065 -0.085 0.062" />
 				<inertia ixx="0.6022" ixy="-0.02364" ixz="-0.1197" iyy="1.7386" iyz="-0.001544" izz="2.0296" />

File: dsr_description/xacro/macro.m1013mobile.blue.xacro (robot description, xacro)
@@ -48,5 +48,5 @@
 		<link name="inertial_link">
 			<inertial>
-				<mass value="346.034" />
+				<mass value="1346.034" />
 				<origin xyz="-0.00065 -0.085 0.062" />
 				<inertia ixx="0.6022" ixy="-0.02364" ixz="-0.1197" iyy="1.7386" iyz="-0.001544" izz="2.0296" />

File: dsr_description/xacro/macro.m1013mobile.white.xacro (robot description, xacro)
@@ -48,5 +48,5 @@
 		<link name="inertial_link">
 			<inertial>
-				<mass value="346.034" />
+				<mass value="1346.034" />
 				<origin xyz="-0.00065 -0.085 0.062" />
 				<inertia ixx="0.6022" ixy="-0.02364" ixz="-0.1197" iyy="1.7386" iyz="-0.001544" izz="2.0296" />

File: dsr_description/xacro/macro.m1509mobile.blue.xacro (robot description, xacro)
@@ -48,5 +48,5 @@
 		<link name="inertial_link">
 			<inertial>
-				<mass value="346.034" />
+				<mass value="1346.034" />
 				<origin xyz="-0.00065 -0.085 0.062" />
 				<inertia ixx="0.6022" ixy="-0.02364" ixz="-0.1197" iyy="1.7386" iyz="-0.001544" izz="2.0296" />

File: dsr_description/xacro/macro.m1509mobile.white.xacro (robot description, xacro)
@@ -48,5 +48,5 @@
 		<link name="inertial_link">
 			<inertial>
-				<mass value="346.034" />
+				<mass value="1346.034" />
 				<origin xyz="-0.00065 -0.085 0.062" />
 				<inertia ixx="0.6022" ixy="-0.02364" ixz="-0.1197" iyy="1.7386" iyz="-0.001544" izz="2.0296" />
