Commit message: update noetic

File: dsr_description/xacro/macro.m1013.white.xacro (robot description, xacro)
@@ -34,4 +34,9 @@
 				<inertia ixx="0.039" ixy="2.1e-05" ixz="-3.61e-05" iyy="0.023" iyz="-0.003" izz="0.039" />
 			</inertial>
+            <collision>
+                <geometry>
+                    <cylinder radius="0.1" length="0.2"/>
+                </geometry>
+            </collision>
 			<visual>
 				<origin rpy="0 0 0" xyz="0 0 0" />
@@ -56,4 +61,10 @@
 				<inertia ixx="0.820" ixy="1.19e-05" ixz="-0.000263" iyy="0.82" iyz="-0.008" izz="0.031" />
 			</inertial>
+            <collision>
+                <origin rpy="0 -1.571 0" xyz="0.3 0 0.1525" />
+                <geometry>
+                    <cylinder radius="0.08" length="0.75"/>
+                </geometry>
+            </collision>
 			<visual>
 				<origin rpy="0 0 0" xyz="0 0 0" />
@@ -112,4 +123,10 @@
 				<inertia ixx="0.177" ixy="-2.34e-06" ixz="-4.92e-06" iyy="0.161" iyz="-0.05" izz="0.022" />
 			</inertial>
+            <collision>
+                <origin rpy="-0.55 0 0" xyz="0 0.07 -0.3" />
+                <geometry>
+                    <cylinder radius="0.07" length="0.4"/>
+                </geometry>
+            </collision>
 			<visual>
 				<origin rpy="0 0 0" xyz="0 0 0" />
@@ -140,4 +157,10 @@
 				<inertia ixx="0.007" ixy="-4.93e-06" ixz="-5.57e-06" iyy="0.004" iyz="-6.64e-05" izz="0.007" />
 			</inertial>
+            <collision>
+                <origin rpy="1.571 0 0" xyz="0 0 0" />
+                <geometry>
+                    <cylinder radius="0.08" length="0.15"/>
+                </geometry>
+            </collision>
 			<visual>
 				<origin rpy="0 0 0" xyz="0 0 0" />

Commit message: update dynamic parameter

File: dsr_description/xacro/macro.m1013.white.xacro (robot description, xacro)
@@ -8,7 +8,9 @@
 		<link name="base_0">
 			<inertial>
-				<mass value="3.722" />
-				<origin xyz="-1.2e-05 -6e-05 0.050723" />
-				<inertia ixx="0.011" ixy="-7.19e-06" ixz="-1.94e-06" iyy="0.011" iyz="4.9e-06" izz="0.014" />
+				<mass value="4.12"/>
+				<origin xyz="-3.4e-05   -0.004815    0.048482"/>
+				<inertia ixx="0.016331" ixy="-6.4837e-06" ixz="2.0048e-06" iyy="0.014945"
+					iyz="-0.00051686"
+					izz="0.022577"/>
 			</inertial>
 			<visual>
@@ -25,12 +27,14 @@
 			<origin rpy="0 0 0" xyz="0 0 0.1525" />
 			<axis xyz="0 0 1" />
-			<limit effort="3460" lower="-6.283" upper="6.283" velocity="2.094" />
+			<limit effort="346" lower="-6.2832" upper="6.2832" velocity="2.0944"/>
 			<dynamics friction="0" />
 		</joint>
 		<link name="link1">
 			<inertial>
-				<mass value="7.446" />
-				<origin xyz="7e-05 0.044281 0.143327" />
-				<inertia ixx="0.039" ixy="2.1e-05" ixz="-3.61e-05" iyy="0.023" iyz="-0.003" izz="0.039" />
+				<mass value="7.8"/>
+				<origin xyz="0.000119      0.0428   -0.006383"/>
+				<inertia ixx="0.04506" ixy="4.1126e-05" ixz="-5.2533e-05" iyy="0.029679"
+					iyz="-0.0019959"
+					izz="0.047056"/>
 			</inertial>
             <collision>
@@ -52,12 +56,14 @@
 			<origin rpy="0 -1.571 -1.571" xyz="0 0.0345 0" />
 			<axis xyz="0 0 1" />
-			<limit effort="3460" lower="-1.658" upper="1.658" velocity="2.094" />
+			<limit effort="346" lower="-6.2832" upper="6.2832" velocity="2.0944"/>
 			<dynamics friction="0" />
 		</joint>
 		<link name="link2">
 			<inertial>
-				<mass value="10.569" />
-				<origin xyz="-1.6e-05 0.189372 0.418558" />
-				<inertia ixx="0.820" ixy="1.19e-05" ixz="-0.000263" iyy="0.82" iyz="-0.008" izz="0.031" />
+				<mass value="10.83"/>
+				<origin xyz="0.25973    -5.3e-05     0.15782"/>
+				<inertia ixx="0.037586" ixy="-0.00036999" ixz="-0.0069927" iyy="0.84943"
+					iyz="4.0201e-05"
+					izz="0.85021"/>
 			</inertial>
             <collision>
@@ -92,14 +98,16 @@
 			<origin rpy="0 0 1.571" xyz="0.62 0 0" />
 			<axis xyz="0 0 1" />
-			<limit effort="1630" lower="-2.356" upper="2.356" velocity="3.142" />
+			<limit effort="163" lower="-2.7925" upper="2.7925" velocity="3.1416"/>
 			<dynamics friction="0" />
 		</joint>
 		<link name="link3">
 			<inertial>
-				<mass value="3.614" />
-				<origin xyz="6e-06 0.07917 0.781807" />
-				<inertia ixx="0.012" ixy="-4.38e-06" ixz="-1.2e-06" iyy="0.008" iyz="0.002" izz="0.011" />
-			</inertial>
-			<visual>
+				<mass value="3.68"/>
+				<origin xyz="-1.5e-05   -0.006702    0.044608"/>
+				<inertia ixx="0.018748" ixy="7.8071e-06" ixz="-5.0324e-06" iyy="0.018972"
+					iyz="-0.00099342"
+					izz="0.011502"/>
+			</inertial>
+            <visual>
 				<origin rpy="0 0 0" xyz="0 0 0" />
 				<geometry>
@@ -114,12 +122,13 @@
 			<origin rpy="1.571 0 0" xyz="0 -0.559 0" />
 			<axis xyz="0 0 1" />
-			<limit effort="50" lower="-6.283" upper="6.283" velocity="3.927" />
+			<limit effort="50" lower="-6.2832" upper="6.2832" velocity="3.927"/>
 			<dynamics friction="0" />
 		</joint>
 		<link name="link4">
 			<inertial>
-				<mass value="3.785" />
-				<origin xyz="-2.1e-05 0.12337 1.148" />
-				<inertia ixx="0.177" ixy="-2.34e-06" ixz="-4.92e-06" iyy="0.161" iyz="-0.05" izz="0.022" />
+				<mass value="3.82"/>
+				<origin xyz="7.1e-05    0.091879    -0.18252"/>
+				<inertia ixx="0.19063" ixy="-1.8037e-05" ixz="-3.8576e-05" iyy="0.17268" iyz="-0.052996"
+					izz="0.030386"/>
 			</inertial>
             <collision>
@@ -148,12 +157,14 @@
 			<origin rpy="-1.571 0 0" xyz="0 0 0" />
 			<axis xyz="0 0 1" />
-			<limit effort="50" lower="-2.356" upper="2.356" velocity="3.927" />
+			<limit effort="50" lower="-6.2832" upper="6.2832" velocity="3.927"/>
 			<dynamics friction="0" />
 		</joint>
 		<link name="link5">
 			<inertial>
-				<mass value="2.598" />
-				<origin xyz="-1.7e-05 0.06662 1.33103" />
-				<inertia ixx="0.007" ixy="-4.93e-06" ixz="-5.57e-06" iyy="0.004" iyz="-6.64e-05" izz="0.007" />
+				<mass value="2.82"/>
+				<origin xyz="-0.000273    0.003651    0.032088"/>
+				<inertia ixx="0.015583" ixy="2.135e-05" ixz="-5.1895e-06" iyy="0.011519"
+					iyz="0.00042553"
+					izz="0.0088671"/>
 			</inertial>
             <collision>
@@ -174,14 +185,16 @@
 			<parent link="link5" />
 			<child link="link6" />
-			<origin rpy="1.571 0 0" xyz="0 -0.121 0" />
-			<axis xyz="0 0 1" />
-			<limit effort="50" lower="-6.283" upper="6.283" velocity="3.927" />
+			<origin rpy="1.571 0 0" xyz="0 -0.124 0" />
+			<axis xyz="0 0 1" />
+			<limit effort="50" lower="-6.2832" upper="6.2832" velocity="3.927"/>
 			<dynamics friction="0" />
 		</joint>
 		<link name="link6">
 			<inertial>
-				<mass value="1.128" />
-				<origin xyz="-0.000174 0.034708 1.40022" />
-				<inertia ixx="0.001" ixy="-2.79e-06" ixz="5.78e-06" iyy="0.001" iyz="-6.67e-06" izz="0.001" />
+				<mass value="1.16"/>
+				<origin xyz="-0.000292       7e-06     -0.0539"/>
+				<inertia ixx="0.0048282" ixy="4.1298e-06" ixz="6.9879e-06" iyy="0.0059519"
+					iyz="4.252e-06"
+					izz="0.0061263"/>
 			</inertial>
 			<visual>
