Commit message: add collision model(cylinder)

File: dsr_description/xacro/macro.m1013.blue.xacro (robot description, xacro)
@@ -34,4 +34,9 @@
 				<inertia ixx="0.039" ixy="2.1e-05" ixz="-3.61e-05" iyy="0.023" iyz="-0.003" izz="0.039" />
 			</inertial>
+            <collision>
+                <geometry>
+                    <cylinder radius="0.1" length="0.2"/>
+                </geometry>
+            </collision>
 			<visual>
 				<origin rpy="0 0 0" xyz="0 0 0" />
@@ -56,4 +61,10 @@
 				<inertia ixx="0.820" ixy="1.19e-05" ixz="-0.000263" iyy="0.82" iyz="-0.008" izz="0.031" />
 			</inertial>
+            <collision>
+                <origin rpy="0 -1.571 0" xyz="0.3 0 0.1525" />
+                <geometry>
+                    <cylinder radius="0.08" length="0.75"/>
+                </geometry>
+            </collision>
 			<visual>
 				<origin rpy="0 0 0" xyz="0 0 0" />
@@ -112,4 +123,10 @@
 				<inertia ixx="0.177" ixy="-2.34e-06" ixz="-4.92e-06" iyy="0.161" iyz="-0.05" izz="0.022" />
 			</inertial>
+            <collision>
+                <origin rpy="-0.55 0 0" xyz="0 0.07 -0.3" />
+                <geometry>
+                    <cylinder radius="0.07" length="0.4"/>
+                </geometry>
+            </collision>
 			<visual>
 				<origin rpy="0 0 0" xyz="0 0 0" />
@@ -140,4 +157,10 @@
 				<inertia ixx="0.007" ixy="-4.93e-06" ixz="-5.57e-06" iyy="0.004" iyz="-6.64e-05" izz="0.007" />
 			</inertial>
+            <collision>
+                <origin rpy="1.571 0 0" xyz="0 0 0" />
+                <geometry>
+                    <cylinder radius="0.08" length="0.15"/>
+                </geometry>
+            </collision>
 			<visual>
 				<origin rpy="0 0 0" xyz="0 0 0" />
@@ -151,5 +174,5 @@
 			<parent link="link5" />
 			<child link="link6" />
-			<origin rpy="1.571 0 0" xyz="0 -0.121 0" />
+			<origin rpy="1.571 0 0" xyz="0 -0.124 0" />
 			<axis xyz="0 0 1" />
 			<limit effort="50" lower="-6.283" upper="6.283" velocity="3.927" />

Commit message: Update macro.m1013.blue.xacro

File: dsr_description/xacro/macro.m1013.blue.xacro (robot description, xacro)
@@ -174,5 +174,5 @@
 			<parent link="link5" />
 			<child link="link6" />
-			<origin rpy="1.571 0 0" xyz="0 -0.124 0" />
+			<origin rpy="1.571 0 0" xyz="0 -0.121 0" />
 			<axis xyz="0 0 1" />
 			<limit effort="50" lower="-6.283" upper="6.283" velocity="3.927" />
