Commit message: Fix collisions in m1509 urdf

File: dsr_description/xacro/macro.m1509.blue.xacro (robot description, xacro)
@@ -1,3 +1,7 @@
 <?xml version="1.0"?>
+<!-- Copy of the xacro from doosan-robots -->
+<!-- @andres.montano: Changed the orientation of the axes so that IKFast works -->
+<!-- @inigo.moreno: Added more collision cillinders -->
+<!-- @inigo.moreno: Limit joints 2, 3 and 5  -->
 <robot name="m1509" xmlns:xacro="http://www.ros.org/wiki/xacro">
 	<xacro:include filename="$(find dsr_description)/config/macro.gazebo.xacro" />
@@ -40,5 +44,5 @@
             <collision>
                 <geometry>
-                    <cylinder radius="0.08" length="0.2"/>
+                    <cylinder radius="0.09" length="0.25"/>
                 </geometry>
             </collision>
@@ -69,7 +73,19 @@
                 <origin rpy="0 -1.571 0" xyz="0.2 0 0.1525" />
                 <geometry>
-                    <cylinder radius="0.08" length="0.5"/>
-                </geometry>
-            </collision>
+                    <cylinder radius="0.09" length="0.5"/>
+                </geometry>
+            </collision>
+			<collision>
+				<origin xyz="0 0 0.16"/>
+				<geometry>
+					<cylinder length=".25" radius=".11"/>
+				</geometry>
+			</collision>
+			<collision>
+				<origin xyz=".41 0 .16"/>
+				<geometry>
+					<cylinder length=".22" radius=".08"/>
+				</geometry>
+			</collision>
 			<visual>
 				<origin rpy="0 0 0" xyz="0 0 0" />
@@ -108,4 +124,10 @@
 					izz="0.011095"/>
 			</inertial>
+			<collision>
+				<origin rpy="1.571 0 0"/>
+				<geometry>
+					<cylinder length=".20" radius=".07"/>
+				</geometry>
+			</collision>
 			<visual>
 				<origin rpy="0 0 0" xyz="0 0 0" />
@@ -135,5 +157,11 @@
                 <origin rpy="-0.55 0 0" xyz="0 0.075 -0.16" />
                 <geometry>
-                    <cylinder radius="0.05" length="0.4"/>
+                    <cylinder radius="0.06" length="0.3"/>
+                </geometry>
+            </collision>
+			<collision>
+				<origin xyz="0 .15 0" rpy="1.571 0 0"/>
+				<geometry>
+					<cylinder length=".19" radius=".07"/>
                 </geometry>
             </collision>
@@ -169,7 +197,7 @@
 			</inertial>
             <collision>
-                <origin rpy="1.571 0 0" xyz="0 0 0" />
-                <geometry>
-                    <cylinder radius="0.06" length="0.15"/>
+                <origin rpy="1.571 0 0" xyz="0 0 0" /> <!-- -0.02 -->
+                <geometry>
+                    <cylinder radius="0.07" length="0.2"/>
                 </geometry>
             </collision>
@@ -198,4 +226,10 @@
 					izz="0.0071373"/>
 			</inertial>
+			<collision>
+				<origin xyz="0 0 -.03"/>
+				<geometry>
+					<cylinder length=".05" radius=".05"/>
+				</geometry>
+			</collision>
 			<visual>
 				<origin rpy="0 0 0" xyz="0 0 0" />

Commit message: Change orientation of joints

File: dsr_description/xacro/macro.m1509.blue.xacro (robot description, xacro)
@@ -54,6 +54,6 @@
 			<parent link="link1" />
 			<child link="link2" />
-			<origin rpy="0 -1.571 -1.571" xyz="0 0.0345 0" />
-			<axis xyz="0 0 1" />
+			<origin rpy="0 0 0" xyz="0 0.0345 0" />
+			<axis xyz="0 1 0" />
 			<limit effort="346" lower="-6.2832" upper="6.2832" velocity="2.618"/>
 			<dynamics friction="0" />
@@ -67,5 +67,5 @@
 			</inertial>
             <collision>
-                <origin rpy="0 -1.571 0" xyz="0.2 0 0.1525" />
+                <origin rpy="0 0 -1.571" xyz="0 0.1525 0.2" />
                 <geometry>
                     <cylinder radius="0.08" length="0.5"/>
@@ -73,5 +73,5 @@
             </collision>
 			<visual>
-				<origin rpy="0 0 0" xyz="0 0 0" />
+				<origin rpy="0 -1.571 -1.571" xyz="0 0 0" />
 				<geometry>
 					<mesh filename="package://dsr_description/meshes/m1509_blue/MF1509_2_0.dae" scale="0.001 0.001 0.001" />
@@ -79,5 +79,5 @@
 			</visual>
 			<visual>
-				<origin rpy="0 0 0" xyz="0 0 0" />
+				<origin rpy="0 -1.571 -1.571" xyz="0 0 0" />
 				<geometry>
 					<mesh filename="package://dsr_description/meshes/m1509_blue/MF1509_2_1.dae" scale="0.001 0.001 0.001" />
@@ -85,5 +85,5 @@
 			</visual>
 			<visual>
-				<origin rpy="0 0 0" xyz="0 0 0" />
+				<origin rpy="0 -1.571 -1.571" xyz="0 0 0" />
 				<geometry>
 					<mesh filename="package://dsr_description/meshes/m1509_blue/MF1509_2_2.dae" scale="0.001 0.001 0.001" />
@@ -95,6 +95,6 @@
 			<parent link="link2" />
 			<child link="link3" />
-			<origin rpy="0 0 1.571" xyz="0.411 0 0" />
-			<axis xyz="0 0 1" />
+			<origin rpy="0 0 0" xyz="0 0 0.411" />
+			<axis xyz="0 1 0" />
 			<limit effort="163" lower="-2.618" upper="2.618" velocity="3.1416"/>
 			<dynamics friction="0" />
@@ -109,5 +109,5 @@
 			</inertial>
 			<visual>
-				<origin rpy="0 0 0" xyz="0 0 0" />
+				<origin rpy="${-pi/2} 0 0" xyz="0 0 0" />
 				<geometry>
 					<mesh filename="package://dsr_description/meshes/m1509_blue/MF1509_3_0.dae" scale="0.001 0.001 0.001" />
@@ -119,5 +119,5 @@
 			<parent link="link3" />
 			<child link="link4" />
-			<origin rpy="1.571 0 0" xyz="0 -0.368 0" />
+			<origin rpy="0 0 0" xyz="0 0 0.368" />
 			<axis xyz="0 0 1" />
 			<limit effort="50" lower="-6.2832" upper="6.2832" velocity="3.927"/>
@@ -155,7 +155,7 @@
 			<parent link="link4" />
 			<child link="link5" />
-			<origin rpy="-1.571 0 0" xyz="0 0 0" />
-			<axis xyz="0 0 1" />
-			<limit effort="50" lower="-6.2832" upper="6.2832" velocity="3.927"/>
+			<origin rpy="0 0 0" xyz="0 0 0" />
+			<axis xyz="0 1 0" />
+			<limit effort="50" lower="-3.1415" upper="3.1415" velocity="3.927"/>
 			<dynamics friction="0" />
 		</joint>
@@ -169,5 +169,5 @@
 			</inertial>
             <collision>
-                <origin rpy="1.571 0 0" xyz="0 0 0" />
+                <origin rpy="0 0 0" xyz="0 0 0" />
                 <geometry>
                     <cylinder radius="0.06" length="0.15"/>
@@ -175,5 +175,5 @@
             </collision>
 			<visual>
-				<origin rpy="0 0 0" xyz="0 0 0" />
+				<origin rpy="-1.571 0 0" xyz="0 0 0" />
 				<geometry>
 					<mesh filename="package://dsr_description/meshes/m1509_blue/MF1509_5_0.dae" scale="0.001 0.001 0.001" />
@@ -185,5 +185,5 @@
 			<parent link="link5" />
 			<child link="link6" />
-			<origin rpy="1.571 0 0" xyz="0 -0.121 0" />
+			<origin rpy="0 0 0" xyz="0 0 0.121" />
 			<axis xyz="0 0 1" />
 			<limit effort="50" lower="-6.2832" upper="6.2832" velocity="3.927"/>
