Commit message: update doosan-ros

File: dsr_description/config/macro.decorations.xacro (robot description, xacro)
@@ -1,4 +1,4 @@
 <?xml version="1.0"?>
-<robot name="dsr_decorations" xmlns:xacro="http://ros.org/wiki/xacro">
+<robot name="dsr_decorations" xmlns:xacro="http://www.ros.org/wiki/xacro">
   <xacro:macro name="mobile_decorate">
     <!-- Spawn chassis -->

File: dsr_description/config/macro.gazebo.xacro (robot description, xacro)
@@ -1,4 +1,4 @@
 <?xml version="1.0"?>
-<robot xmlns:xacro="http://ros.org/wiki/xacro">
+<robot xmlns:xacro="http://www.ros.org/wiki/xacro">
 	<xacro:macro name="dsr_gazebo" params="namespace:=/">
 		<!-- Base -->

File: dsr_description/config/macro.materials.xacro (robot description, xacro)
@@ -1,4 +1,4 @@
 <?xml version="1.0"?>
-<robot name="dsr_materials" xmlns:xacro="http://ros.org/wiki/xacro">
+<robot name="dsr_materials" xmlns:xacro="http://www.ros.org/wiki/xacro">
 	<xacro:macro name="dsr_materials">
 		<material name="black">

File: dsr_description/config/macro.transmission.xacro (robot description, xacro)
@@ -1,4 +1,4 @@
 <?xml version="1.0"?>
-<robot xmlns:xacro="http://ros.org/wiki/xacro">
+<robot xmlns:xacro="http://www.ros.org/wiki/xacro">
 	<xacro:macro name="dsr_transmission">
 		<!-- Transmission 1 -->

File: dsr_description/config/macro.wheel.xacro (robot description, xacro)
@@ -1,4 +1,4 @@
 <?xml version="1.0"?>
-<robot xmlns:xacro="http://ros.org/wiki/xacro" name="mobile_wheel">
+<robot xmlns:xacro="http://www.ros.org/wiki/xacro" name="mobile_wheel">
 	<xacro:macro name="mobile_wheel" params="wheel_prefix *joint_pose">
 		<link name="${wheel_prefix}_wheel_link">

File: dsr_description/xacro/m0609.urdf.xacro (robot description, xacro)
@@ -1,4 +1,4 @@
 <?xml version="1.0"?>
-<robot xmlns:xacro="http://ros.org/wiki/xacro" name="m0609" >
+<robot xmlns:xacro="http://www.ros.org/wiki/xacro" name="m0609" >
   <xacro:arg name="color"   default="white"/>
   <xacro:arg name="gripper" default="none"/>
@@ -11,9 +11,9 @@
      <xacro:include filename="$(find dsr_description)/xacro/macro.m0609.blue.xacro" />
   </xacro:if>
+  <xacro:m0609 namespace="$(arg namespace)"/>
+  <link name="world" />
   <xacro:if value="${gr == 'robotiq_2f'}">
      <xacro:include filename="$(find dsr_description)/xacro/robotiq_2f.urdf.xacro" />
   </xacro:if>
-  <xacro:m0609 namespace="$(arg namespace)"/>
-  <link name="world" />
   <!-- World fixed joint-->
   <joint name="world_fixed" type="fixed">

File: dsr_description/xacro/m0609mobile.urdf.xacro (robot description, xacro)
@@ -1,4 +1,4 @@
 <?xml version="1.0"?>
-<robot xmlns:xacro="http://ros.org/wiki/xacro" name="m0609mobile" >
+<robot xmlns:xacro="http://www.ros.org/wiki/xacro" name="m0609mobile" >
   <xacro:arg name="color"   default="white"/>
   <xacro:arg name="gripper" default="none"/>
@@ -11,4 +11,7 @@
     <xacro:include filename="$(find dsr_description)/xacro/macro.m0609mobile.blue.xacro" />
   </xacro:if>
+  <xacro:if value="${gr == 'robotiq_2f'}">
+     <xacro:include filename="$(find dsr_description)/xacro/robotiq_2f.urdf.xacro" />
+  </xacro:if>
   <xacro:m0609mobile namespace="$(arg namespace)"/>
 </robot>

File: dsr_description/xacro/m0617.urdf.xacro (robot description, xacro)
@@ -1,4 +1,4 @@
 <?xml version="1.0"?>
-<robot xmlns:xacro="http://ros.org/wiki/xacro" name="m0617" >
+<robot xmlns:xacro="http://www.ros.org/wiki/xacro" name="m0617" >
   <xacro:arg name="color"   default="white"/>
   <xacro:arg name="gripper" default="none"/>

File: dsr_description/xacro/m0617mobile.urdf.xacro (robot description, xacro)
@@ -1,4 +1,4 @@
 <?xml version="1.0"?>
-<robot xmlns:xacro="http://ros.org/wiki/xacro" name="m0617mobile" >
+<robot xmlns:xacro="http://www.ros.org/wiki/xacro" name="m0617mobile" >
   <xacro:arg name="color"   default="white"/>
   <xacro:arg name="gripper" default="none"/>
@@ -11,4 +11,7 @@
     <xacro:include filename="$(find dsr_description)/xacro/macro.m0617mobile.blue.xacro" />
   </xacro:if>
+  <xacro:if value="${gr == 'robotiq_2f'}">
+     <xacro:include filename="$(find dsr_description)/xacro/robotiq_2f.urdf.xacro" />
+  </xacro:if>
   <xacro:m0617mobile namespace="$(arg namespace)"/>
 </robot>

File: dsr_description/xacro/m1013.urdf.xacro (robot description, xacro)
@@ -1,4 +1,4 @@
 <?xml version="1.0"?>
-<robot xmlns:xacro="http://ros.org/wiki/xacro" name="m1013" >
+<robot xmlns:xacro="http://www.ros.org/wiki/xacro" name="m1013" >
   <xacro:arg name="color"   default="white"/>
   <xacro:arg name="gripper" default="none"/>
@@ -11,9 +11,9 @@
      <xacro:include filename="$(find dsr_description)/xacro/macro.m1013.blue.xacro" />
   </xacro:if>
+  <xacro:m1013 namespace="$(arg namespace)"/>
+  <link name="world" />
   <xacro:if value="${gr == 'robotiq_2f'}">
      <xacro:include filename="$(find dsr_description)/xacro/robotiq_2f.urdf.xacro" />
   </xacro:if>
-  <xacro:m1013 namespace="$(arg namespace)"/>
-  <link name="world" />
   <!-- World fixed joint-->
   <joint name="world_fixed" type="fixed">

File: dsr_description/xacro/m1013mobile.urdf.xacro (robot description, xacro)
@@ -1,4 +1,4 @@
 <?xml version="1.0"?>
-<robot xmlns:xacro="http://ros.org/wiki/xacro" name="m1013mobile" >
+<robot xmlns:xacro="http://www.ros.org/wiki/xacro" name="m1013mobile" >
   <xacro:arg name="color"   default="white"/>
   <xacro:arg name="gripper" default="none"/>
@@ -11,4 +11,7 @@
     <xacro:include filename="$(find dsr_description)/xacro/macro.m1013mobile.blue.xacro" />
   </xacro:if>
+  <xacro:if value="${gr == 'robotiq_2f'}">
+     <xacro:include filename="$(find dsr_description)/xacro/robotiq_2f.urdf.xacro" />
+  </xacro:if>
   <xacro:m1013mobile namespace="$(arg namespace)"/>
 </robot>

File: dsr_description/xacro/m1509.urdf.xacro (robot description, xacro)
@@ -1,4 +1,4 @@
 <?xml version="1.0"?>
-<robot xmlns:xacro="http://ros.org/wiki/xacro" name="m1509" >
+<robot xmlns:xacro="http://www.ros.org/wiki/xacro" name="m1509" >
   <xacro:arg name="color"   default="white"/>
   <xacro:arg name="gripper" default="none"/>
@@ -11,9 +11,9 @@
      <xacro:include filename="$(find dsr_description)/xacro/macro.m1509.blue.xacro" />
   </xacro:if>
+  <xacro:m1509 namespace="$(arg namespace)"/>
+  <link name="world" />
   <xacro:if value="${gr == 'robotiq_2f'}">
      <xacro:include filename="$(find dsr_description)/xacro/robotiq_2f.urdf.xacro" />
   </xacro:if>
-  <xacro:m1509 namespace="$(arg namespace)"/>
-  <link name="world" />
   <!-- World fixed joint-->
   <joint name="world_fixed" type="fixed">

File: dsr_description/xacro/m1509mobile.urdf.xacro (robot description, xacro)
@@ -1,4 +1,4 @@
 <?xml version="1.0"?>
-<robot xmlns:xacro="http://ros.org/wiki/xacro" name="m1509mobile" >
+<robot xmlns:xacro="http://www.ros.org/wiki/xacro" name="m1509mobile" >
   <xacro:arg name="color"   default="white"/>
   <xacro:arg name="gripper" default="none"/>
@@ -11,4 +11,7 @@
     <xacro:include filename="$(find dsr_description)/xacro/macro.m1509mobile.blue.xacro" />
   </xacro:if>
+  <xacro:if value="${gr == 'robotiq_2f'}">
+     <xacro:include filename="$(find dsr_description)/xacro/robotiq_2f.urdf.xacro" />
+  </xacro:if>
   <xacro:m1509mobile namespace="$(arg namespace)"/>
 </robot>

File: dsr_description/xacro/macro.m0609.blue.xacro (robot description, xacro)
@@ -1,4 +1,4 @@
 <?xml version="1.0"?>
-<robot name="m0609" xmlns:xacro="http://ros.org/wiki/xacro">
+<robot name="m0609" xmlns:xacro="http://www.ros.org/wiki/xacro">
 	<xacro:include filename="$(find dsr_description)/config/macro.gazebo.xacro" />
 	<xacro:include filename="$(find dsr_description)/config/macro.transmission.xacro" />

File: dsr_description/xacro/macro.m0609.white.xacro (robot description, xacro)
@@ -1,4 +1,4 @@
 <?xml version="1.0"?>
-<robot name="m0609" xmlns:xacro="http://ros.org/wiki/xacro">
+<robot name="m0609" xmlns:xacro="http://www.ros.org/wiki/xacro">
 	<xacro:include filename="$(find dsr_description)/config/macro.gazebo.xacro" />
 	<xacro:include filename="$(find dsr_description)/config/macro.transmission.xacro" />

File: dsr_description/xacro/macro.m0609mobile.blue.xacro (robot description, xacro)
@@ -1,4 +1,4 @@
 <?xml version="1.0"?>
-<robot name="m0609mobile" xmlns:xacro="http://ros.org/wiki/xacro">
+<robot name="m0609mobile" xmlns:xacro="http://www.ros.org/wiki/xacro">
 	<xacro:include filename="$(find dsr_description)/config/macro.decorations.xacro" />
 	<xacro:include filename="$(find dsr_description)/config/macro.wheel.xacro" />

File: dsr_description/xacro/macro.m0609mobile.white.xacro (robot description, xacro)
@@ -1,4 +1,4 @@
 <?xml version="1.0"?>
-<robot name="m0609mobile" xmlns:xacro="http://ros.org/wiki/xacro">
+<robot name="m0609mobile" xmlns:xacro="http://www.ros.org/wiki/xacro">
 	<xacro:include filename="$(find dsr_description)/config/macro.decorations.xacro" />
 	<xacro:include filename="$(find dsr_description)/config/macro.wheel.xacro" />

File: dsr_description/xacro/macro.m0617.blue.xacro (robot description, xacro)
@@ -1,4 +1,4 @@
 <?xml version="1.0"?>
-<robot name="m0617" xmlns:xacro="http://ros.org/wiki/xacro">
+<robot name="m0617" xmlns:xacro="http://www.ros.org/wiki/xacro">
 	<xacro:include filename="$(find dsr_description)/config/macro.gazebo.xacro" />
 	<xacro:include filename="$(find dsr_description)/config/macro.transmission.xacro" />

File: dsr_description/xacro/macro.m0617.white.xacro (robot description, xacro)
@@ -1,4 +1,4 @@
 <?xml version="1.0"?>
-<robot name="m0617" xmlns:xacro="http://ros.org/wiki/xacro">
+<robot name="m0617" xmlns:xacro="http://www.ros.org/wiki/xacro">
 	<xacro:include filename="$(find dsr_description)/config/macro.gazebo.xacro" />
 	<xacro:include filename="$(find dsr_description)/config/macro.transmission.xacro" />

File: dsr_description/xacro/macro.m0617mobile.blue.xacro (robot description, xacro)
@@ -1,4 +1,4 @@
 <?xml version="1.0"?>
-<robot name="m0617mobile" xmlns:xacro="http://ros.org/wiki/xacro">
+<robot name="m0617mobile" xmlns:xacro="http://www.ros.org/wiki/xacro">
 	<xacro:include filename="$(find dsr_description)/config/macro.decorations.xacro" />
 	<xacro:include filename="$(find dsr_description)/config/macro.wheel.xacro" />
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