Commit message: add collision model(cylinder)

File: dsr_description/config/macro.gazebo.xacro (robot description, xacro)
@@ -3,5 +3,10 @@
 	<xacro:macro name="dsr_gazebo" params="namespace:=/">
 		<!-- Base -->
+        <selfCollide>true</selfCollide>
+        <gazebo reference="dsr01">
+            <selfCollide>true</selfCollide>
+        </gazebo>
 		<gazebo reference="base_0">
+            <selfCollide>true</selfCollide>
 			<kp>1000000.0</kp>
 			<kd>100.0</kd>
@@ -13,4 +18,5 @@
 		<!-- Link1 -->
 		<gazebo reference="link1">
+            <selfCollide>true</selfCollide>
 			<kp>1000000.0</kp>
 			<kd>100.0</kd>
@@ -22,4 +28,5 @@
 		<!-- Link2 -->
 		<gazebo reference="link2">
+            <selfCollide>true</selfCollide>
 			<kp>1000000.0</kp>
 			<kd>100.0</kd>
@@ -31,4 +38,5 @@
 		<!-- Link3 -->
 		<gazebo reference="link3">
+            <selfCollide>true</selfCollide>
 			<kp>1000000.0</kp>
 			<kd>100.0</kd>
@@ -40,4 +48,5 @@
 		<!-- Link4 -->
 		<gazebo reference="link4">
+            <selfCollide>true</selfCollide>
 			<kp>1000000.0</kp>
 			<kd>100.0</kd>
@@ -49,4 +58,5 @@
 		<!-- Link5 -->
 		<gazebo reference="link5">
+            <selfCollide>true</selfCollide>
 			<kp>1000000.0</kp>
 			<kd>100.0</kd>
@@ -58,4 +68,5 @@
 		<!-- Link6 -->
 		<gazebo reference="link6">
+            <selfCollide>true</selfCollide>
 			<kp>1000000.0</kp>
 			<kd>100.0</kd>
@@ -67,4 +78,5 @@
 		<!-- ros_control plugin -->
 		<gazebo>
+            <selfCollide>true</selfCollide>
 			<plugin name="gazebo_ros_control" filename="libgazebo_ros_control.so">
 				<robotNamespace>/${namespace}</robotNamespace>

File: dsr_description/xacro/macro.a0509.blue.xacro (robot description, xacro)
@@ -34,4 +34,9 @@
 				<inertia ixx="0.039" ixy="2.1e-05" ixz="-3.61e-05" iyy="0.023" iyz="-0.003" izz="0.039" />
 			</inertial>
+            <collision>
+                <geometry>
+                    <cylinder radius="0.08" length="0.2"/>
+                </geometry>
+            </collision>
 			<visual>
 				<origin rpy="0 0 0" xyz="0 0 0" />
@@ -68,4 +73,10 @@
 				<inertia ixx="0.820" ixy="1.19e-05" ixz="-0.000263" iyy="0.82" iyz="-0.008" izz="0.031" />
 			</inertial>
+            <collision>
+                <origin rpy="0 -1.571 0" xyz="0.2 0 0.1525" />
+                <geometry>
+                    <cylinder radius="0.08" length="0.5"/>
+                </geometry>
+            </collision>
 			<visual>
 				<origin rpy="0 0 0" xyz="0 0 0" />
@@ -130,4 +141,10 @@
 				<inertia ixx="0.177" ixy="-2.34e-06" ixz="-4.92e-06" iyy="0.161" iyz="-0.05" izz="0.022" />
 			</inertial>
+            <collision>
+                <origin rpy="-0.55 0 0" xyz="0 0.05 -0.2" />
+                <geometry>
+                    <cylinder radius="0.05" length="0.4"/>
+                </geometry>
+            </collision>
 			<visual>
 				<origin rpy="0 0 0" xyz="0 0 0" />
@@ -158,4 +175,10 @@
 				<inertia ixx="0.007" ixy="-4.93e-06" ixz="-5.57e-06" iyy="0.004" iyz="-6.64e-05" izz="0.007" />
 			</inertial>
+            <collision>
+                <origin rpy="1.571 0 0" xyz="0 0 0" />
+                <geometry>
+                    <cylinder radius="0.06" length="0.15"/>
+                </geometry>
+            </collision>
 			<visual>
 				<origin rpy="0 0 0" xyz="0 0 0" />

File: dsr_description/xacro/macro.a0509.white.xacro (robot description, xacro)
@@ -34,4 +34,9 @@
 				<inertia ixx="0.039" ixy="2.1e-05" ixz="-3.61e-05" iyy="0.023" iyz="-0.003" izz="0.039" />
 			</inertial>
+            <collision>
+                <geometry>
+                    <cylinder radius="0.08" length="0.2"/>
+                </geometry>
+            </collision>
 			<visual>
 				<origin rpy="0 0 0" xyz="0 0 0" />
@@ -68,4 +73,10 @@
 				<inertia ixx="0.820" ixy="1.19e-05" ixz="-0.000263" iyy="0.82" iyz="-0.008" izz="0.031" />
 			</inertial>
+            <collision>
+                <origin rpy="0 -1.571 0" xyz="0.2 0 0.1525" />
+                <geometry>
+                    <cylinder radius="0.08" length="0.5"/>
+                </geometry>
+            </collision>
 			<visual>
 				<origin rpy="0 0 0" xyz="0 0 0" />
@@ -130,4 +141,10 @@
 				<inertia ixx="0.177" ixy="-2.34e-06" ixz="-4.92e-06" iyy="0.161" iyz="-0.05" izz="0.022" />
 			</inertial>
+            <collision>
+                <origin rpy="-0.55 0 0" xyz="0 0.05 -0.2" />
+                <geometry>
+                    <cylinder radius="0.05" length="0.4"/>
+                </geometry>
+            </collision>
 			<visual>
 				<origin rpy="0 0 0" xyz="0 0 0" />
@@ -158,4 +175,10 @@
 				<inertia ixx="0.007" ixy="-4.93e-06" ixz="-5.57e-06" iyy="0.004" iyz="-6.64e-05" izz="0.007" />
 			</inertial>
+            <collision>
+                <origin rpy="1.571 0 0" xyz="0 0 0" />
+                <geometry>
+                    <cylinder radius="0.06" length="0.15"/>
+                </geometry>
+            </collision>
 			<visual>
 				<origin rpy="0 0 0" xyz="0 0 0" />

File: dsr_description/xacro/macro.a0912.blue.xacro (robot description, xacro)
@@ -34,4 +34,9 @@
 				<inertia ixx="0.039" ixy="2.1e-05" ixz="-3.61e-05" iyy="0.023" iyz="-0.003" izz="0.039" />
 			</inertial>
+            <collision>
+                <geometry>
+                    <cylinder radius="0.08" length="0.2"/>
+                </geometry>
+            </collision>
 			<visual>
 				<origin rpy="0 0 0" xyz="0 0 0" />
@@ -68,4 +73,10 @@
 				<inertia ixx="0.820" ixy="1.19e-05" ixz="-0.000263" iyy="0.82" iyz="-0.008" izz="0.031" />
 			</inertial>
+            <collision>
+                <origin rpy="0 -1.571 0" xyz="0.3 0 0.1525" />
+                <geometry>
+                    <cylinder radius="0.08" length="0.6"/>
+                </geometry>
+            </collision>
 			<visual>
 				<origin rpy="0 0 0" xyz="0 0 0" />
@@ -130,4 +141,10 @@
 				<inertia ixx="0.177" ixy="-2.34e-06" ixz="-4.92e-06" iyy="0.161" iyz="-0.05" izz="0.022" />
 			</inertial>
+            <collision>
+                <origin rpy="-0.46 0 0" xyz="0 0.075 -0.2" />
+                <geometry>
+                    <cylinder radius="0.05" length="0.4"/>
+                </geometry>
+            </collision>
 			<visual>
 				<origin rpy="0 0 0" xyz="0 0 0" />
@@ -158,4 +175,10 @@
 				<inertia ixx="0.007" ixy="-4.93e-06" ixz="-5.57e-06" iyy="0.004" iyz="-6.64e-05" izz="0.007" />
 			</inertial>
+            <collision>
+                <origin rpy="1.571 0 0" xyz="0 0 0" />
+                <geometry>
+                    <cylinder radius="0.06" length="0.15"/>
+                </geometry>
+            </collision>
 			<visual>
 				<origin rpy="0 0 0" xyz="0 0 0" />

File: dsr_description/xacro/macro.a0912.white.xacro (robot description, xacro)
@@ -34,4 +34,9 @@
 				<inertia ixx="0.039" ixy="2.1e-05" ixz="-3.61e-05" iyy="0.023" iyz="-0.003" izz="0.039" />
 			</inertial>
+            <collision>
+                <geometry>
+                    <cylinder radius="0.08" length="0.2"/>
+                </geometry>
+            </collision>
 			<visual>
 				<origin rpy="0 0 0" xyz="0 0 0" />
@@ -68,4 +73,10 @@
 				<inertia ixx="0.820" ixy="1.19e-05" ixz="-0.000263" iyy="0.82" iyz="-0.008" izz="0.031" />
 			</inertial>
+            <collision>
+                <origin rpy="0 -1.571 0" xyz="0.3 0 0.1525" />
+                <geometry>
+                    <cylinder radius="0.08" length="0.6"/>
+                </geometry>
+            </collision>
 			<visual>
 				<origin rpy="0 0 0" xyz="0 0 0" />
@@ -130,4 +141,10 @@
 				<inertia ixx="0.177" ixy="-2.34e-06" ixz="-4.92e-06" iyy="0.161" iyz="-0.05" izz="0.022" />
 			</inertial>
+            <collision>
+                <origin rpy="-0.46 0 0" xyz="0 0.075 -0.2" />
+                <geometry>
+                    <cylinder radius="0.05" length="0.4"/>
+                </geometry>
+            </collision>
 			<visual>
 				<origin rpy="0 0 0" xyz="0 0 0" />
@@ -158,4 +175,10 @@
 				<inertia ixx="0.007" ixy="-4.93e-06" ixz="-5.57e-06" iyy="0.004" iyz="-6.64e-05" izz="0.007" />
 			</inertial>
+            <collision>
+                <origin rpy="1.571 0 0" xyz="0 0 0" />
+                <geometry>
+                    <cylinder radius="0.06" length="0.15"/>
+                </geometry>
+            </collision>
 			<visual>
 				<origin rpy="0 0 0" xyz="0 0 0" />

File: dsr_description/xacro/macro.m0609.blue.xacro (robot description, xacro)
@@ -34,4 +34,9 @@
 				<inertia ixx="0.039" ixy="2.1e-05" ixz="-3.61e-05" iyy="0.023" iyz="-0.003" izz="0.039" />
 			</inertial>
+            <collision>
+                <geometry>
+                    <cylinder radius="0.08" length="0.2"/>
+                </geometry>
+            </collision>
 			<visual>
 				<origin rpy="0 0 0" xyz="0 0 0" />
@@ -56,4 +61,10 @@
 				<inertia ixx="0.820" ixy="1.19e-05" ixz="-0.000263" iyy="0.82" iyz="-0.008" izz="0.031" />
 			</inertial>
+            <collision>
+                <origin rpy="0 -1.571 0" xyz="0.2 0 0.1525" />
+                <geometry>
+                    <cylinder radius="0.08" length="0.5"/>
+                </geometry>
+            </collision>
 			<visual>
 				<origin rpy="0 0 0" xyz="0 0 0" />
@@ -112,4 +123,10 @@
 				<inertia ixx="0.177" ixy="-2.34e-06" ixz="-4.92e-06" iyy="0.161" iyz="-0.05" izz="0.022" />
 			</inertial>
+            <collision>
+                <origin rpy="-0.55 0 0" xyz="0 0.075 -0.16" />
+                <geometry>
+                    <cylinder radius="0.05" length="0.4"/>
+                </geometry>
+            </collision>
 			<visual>
 				<origin rpy="0 0 0" xyz="0 0 0" />
@@ -140,4 +157,10 @@
 				<inertia ixx="0.007" ixy="-4.93e-06" ixz="-5.57e-06" iyy="0.004" iyz="-6.64e-05" izz="0.007" />
 			</inertial>
+            <collision>
+                <origin rpy="1.571 0 0" xyz="0 0 0" />
+                <geometry>
+                    <cylinder radius="0.06" length="0.15"/>
+                </geometry>
+            </collision>
 			<visual>
 				<origin rpy="0 0 0" xyz="0 0 0" />

File: dsr_description/xacro/macro.m0609.white.xacro (robot description, xacro)
@@ -34,4 +34,9 @@
 				<inertia ixx="0.039" ixy="2.1e-05" ixz="-3.61e-05" iyy="0.023" iyz="-0.003" izz="0.039" />
 			</inertial>
+            <collision>
+                <geometry>
+                    <cylinder radius="0.08" length="0.2"/>
+                </geometry>
+            </collision>
 			<visual>
 				<origin rpy="0 0 0" xyz="0 0 0" />
@@ -56,4 +61,10 @@
 				<inertia ixx="0.820" ixy="1.19e-05" ixz="-0.000263" iyy="0.82" iyz="-0.008" izz="0.031" />
 			</inertial>
+            <collision>
+                <origin rpy="0 -1.571 0" xyz="0.2 0 0.1525" />
+                <geometry>
+                    <cylinder radius="0.08" length="0.5"/>
+                </geometry>
+            </collision>
 			<visual>
 				<origin rpy="0 0 0" xyz="0 0 0" />
@@ -112,4 +123,10 @@
 				<inertia ixx="0.177" ixy="-2.34e-06" ixz="-4.92e-06" iyy="0.161" iyz="-0.05" izz="0.022" />
 			</inertial>
+            <collision>
+                <origin rpy="-0.55 0 0" xyz="0 0.075 -0.16" />
+                <geometry>
+                    <cylinder radius="0.05" length="0.4"/>
+                </geometry>
+            </collision>
 			<visual>
 				<origin rpy="0 0 0" xyz="0 0 0" />
@@ -140,4 +157,10 @@
 				<inertia ixx="0.007" ixy="-4.93e-06" ixz="-5.57e-06" iyy="0.004" iyz="-6.64e-05" izz="0.007" />
 			</inertial>
+            <collision>
+                <origin rpy="1.571 0 0" xyz="0 0 0" />
+                <geometry>
+                    <cylinder radius="0.06" length="0.15"/>
+                </geometry>
+            </collision>
 			<visual>
 				<origin rpy="0 0 0" xyz="0 0 0" />

File: dsr_description/xacro/macro.m0617.blue.xacro (robot description, xacro)
@@ -34,4 +34,9 @@
 				<inertia ixx="0.039" ixy="2.1e-05" ixz="-3.61e-05" iyy="0.023" iyz="-0.003" izz="0.039" />
 			</inertial>
+            <collision>
+                <geometry>
+                    <cylinder radius="0.1" length="0.2"/>
+                </geometry>
+            </collision>
 			<visual>
 				<origin rpy="0 0 0" xyz="0 0 0" />
@@ -56,4 +61,10 @@
 				<inertia ixx="0.820" ixy="1.19e-05" ixz="-0.000263" iyy="0.82" iyz="-0.008" izz="0.031" />
 			</inertial>
+            <collision>
+                <origin rpy="0 -1.571 0" xyz="0.45 0 0.1525" />
+                <geometry>
+                    <cylinder radius="0.08" length="0.9"/>
+                </geometry>
+            </collision>
 			<visual>
 				<origin rpy="0 0 0" xyz="0 0 0" />
@@ -112,4 +123,10 @@
 				<inertia ixx="0.177" ixy="-2.34e-06" ixz="-4.92e-06" iyy="0.161" iyz="-0.05" izz="0.022" />
 			</inertial>
+            <collision>
+                <origin rpy="-0.32 0 0" xyz="0 0.07 -0.32" />
+                <geometry>
+                    <cylinder radius="0.07" length="0.5"/>
+                </geometry>
+            </collision>
 			<visual>
 				<origin rpy="0 0 0" xyz="0 0 0" />
@@ -140,4 +157,10 @@
 				<inertia ixx="0.007" ixy="-4.93e-06" ixz="-5.57e-06" iyy="0.004" iyz="-6.64e-05" izz="0.007" />
 			</inertial>
+            <collision>
+                <origin rpy="1.571 0 0" xyz="0 0 0" />
+                <geometry>
+                    <cylinder radius="0.08" length="0.15"/>
+                </geometry>
+            </collision>
 			<visual>
 				<origin rpy="0 0 0" xyz="0 0 0" />

File: dsr_description/xacro/macro.m0617.white.xacro (robot description, xacro)
@@ -34,4 +34,9 @@
 				<inertia ixx="0.039" ixy="2.1e-05" ixz="-3.61e-05" iyy="0.023" iyz="-0.003" izz="0.039" />
 			</inertial>
+            <collision>
+                <geometry>
+                    <cylinder radius="0.1" length="0.2"/>
+                </geometry>
+            </collision>
 			<visual>
 				<origin rpy="0 0 0" xyz="0 0 0" />
@@ -56,4 +61,10 @@
 				<inertia ixx="0.820" ixy="1.19e-05" ixz="-0.000263" iyy="0.82" iyz="-0.008" izz="0.031" />
 			</inertial>
+            <collision>
+                <origin rpy="0 -1.571 0" xyz="0.45 0 0.1525" />
+                <geometry>
+                    <cylinder radius="0.08" length="0.9"/>
+                </geometry>
+            </collision>
 			<visual>
 				<origin rpy="0 0 0" xyz="0 0 0" />
@@ -112,4 +123,10 @@
 				<inertia ixx="0.177" ixy="-2.34e-06" ixz="-4.92e-06" iyy="0.161" iyz="-0.05" izz="0.022" />
 			</inertial>
+            <collision>
+                <origin rpy="-0.32 0 0" xyz="0 0.07 -0.32" />
+                <geometry>
+                    <cylinder radius="0.07" length="0.5"/>
+                </geometry>
+            </collision>
 			<visual>
 				<origin rpy="0 0 0" xyz="0 0 0" />
@@ -140,4 +157,10 @@
 				<inertia ixx="0.007" ixy="-4.93e-06" ixz="-5.57e-06" iyy="0.004" iyz="-6.64e-05" izz="0.007" />
 			</inertial>
+            <collision>
+                <origin rpy="1.571 0 0" xyz="0 0 0" />
+                <geometry>
+                    <cylinder radius="0.08" length="0.15"/>
+                </geometry>
+            </collision>
 			<visual>
 				<origin rpy="0 0 0" xyz="0 0 0" />

File: dsr_description/xacro/macro.m1013.blue.xacro (robot description, xacro)
@@ -34,4 +34,9 @@
 				<inertia ixx="0.039" ixy="2.1e-05" ixz="-3.61e-05" iyy="0.023" iyz="-0.003" izz="0.039" />
 			</inertial>
+            <collision>
+                <geometry>
+                    <cylinder radius="0.1" length="0.2"/>
+                </geometry>
+            </collision>
 			<visual>
 				<origin rpy="0 0 0" xyz="0 0 0" />
@@ -56,4 +61,10 @@
 				<inertia ixx="0.820" ixy="1.19e-05" ixz="-0.000263" iyy="0.82" iyz="-0.008" izz="0.031" />
 			</inertial>
+            <collision>
+                <origin rpy="0 -1.571 0" xyz="0.3 0 0.1525" />
+                <geometry>
+                    <cylinder radius="0.08" length="0.75"/>
+                </geometry>
+            </collision>
 			<visual>
 				<origin rpy="0 0 0" xyz="0 0 0" />
@@ -112,4 +123,10 @@
 				<inertia ixx="0.177" ixy="-2.34e-06" ixz="-4.92e-06" iyy="0.161" iyz="-0.05" izz="0.022" />
 			</inertial>
+            <collision>
+                <origin rpy="-0.55 0 0" xyz="0 0.07 -0.3" />
+                <geometry>
+                    <cylinder radius="0.07" length="0.4"/>
+                </geometry>
+            </collision>
 			<visual>
 				<origin rpy="0 0 0" xyz="0 0 0" />
@@ -140,4 +157,10 @@
 				<inertia ixx="0.007" ixy="-4.93e-06" ixz="-5.57e-06" iyy="0.004" iyz="-6.64e-05" izz="0.007" />
 			</inertial>
+            <collision>
+                <origin rpy="1.571 0 0" xyz="0 0 0" />
+                <geometry>
+                    <cylinder radius="0.08" length="0.15"/>
+                </geometry>
+            </collision>
 			<visual>
 				<origin rpy="0 0 0" xyz="0 0 0" />

File: dsr_description/xacro/macro.m1013.white.xacro (robot description, xacro)
@@ -34,4 +34,9 @@
 				<inertia ixx="0.039" ixy="2.1e-05" ixz="-3.61e-05" iyy="0.023" iyz="-0.003" izz="0.039" />
 			</inertial>
+            <collision>
+                <geometry>
+                    <cylinder radius="0.1" length="0.2"/>
+                </geometry>
+            </collision>
 			<visual>
 				<origin rpy="0 0 0" xyz="0 0 0" />
@@ -56,4 +61,10 @@
 				<inertia ixx="0.820" ixy="1.19e-05" ixz="-0.000263" iyy="0.82" iyz="-0.008" izz="0.031" />
 			</inertial>
+            <collision>
+                <origin rpy="0 -1.571 0" xyz="0.3 0 0.1525" />
+                <geometry>
+                    <cylinder radius="0.08" length="0.75"/>
+                </geometry>
+            </collision>
 			<visual>
 				<origin rpy="0 0 0" xyz="0 0 0" />
@@ -90,5 +101,5 @@
 				<inertia ixx="0.012" ixy="-4.38e-06" ixz="-1.2e-06" iyy="0.008" iyz="0.002" izz="0.011" />
 			</inertial>
-			<visual>
+            <visual>
 				<origin rpy="0 0 0" xyz="0 0 0" />
 				<geometry>
@@ -112,4 +123,10 @@
 				<inertia ixx="0.177" ixy="-2.34e-06" ixz="-4.92e-06" iyy="0.161" iyz="-0.05" izz="0.022" />
 			</inertial>
+            <collision>
+                <origin rpy="-0.55 0 0" xyz="0 0.07 -0.3" />
+                <geometry>
+                    <cylinder radius="0.07" length="0.4"/>
+                </geometry>
+            </collision>
 			<visual>
 				<origin rpy="0 0 0" xyz="0 0 0" />
@@ -140,4 +157,10 @@
 				<inertia ixx="0.007" ixy="-4.93e-06" ixz="-5.57e-06" iyy="0.004" iyz="-6.64e-05" izz="0.007" />
 			</inertial>
+            <collision>
+                <origin rpy="1.571 0 0" xyz="0 0 0" />
+                <geometry>
+                    <cylinder radius="0.08" length="0.15"/>
+                </geometry>
+            </collision>
 			<visual>
 				<origin rpy="0 0 0" xyz="0 0 0" />

File: dsr_description/xacro/macro.m1509.blue.xacro (robot description, xacro)
@@ -34,4 +34,9 @@
 				<inertia ixx="0.039" ixy="2.1e-05" ixz="-3.61e-05" iyy="0.023" iyz="-0.003" izz="0.039" />
 			</inertial>
+            <collision>
+                <geometry>
+                    <cylinder radius="0.08" length="0.2"/>
+                </geometry>
+            </collision>
 			<visual>
 				<origin rpy="0 0 0" xyz="0 0 0" />
@@ -56,4 +61,10 @@
 				<inertia ixx="0.820" ixy="1.19e-05" ixz="-0.000263" iyy="0.82" iyz="-0.008" izz="0.031" />
 			</inertial>
+            <collision>
+                <origin rpy="0 -1.571 0" xyz="0.2 0 0.1525" />
+                <geometry>
+                    <cylinder radius="0.08" length="0.5"/>
+                </geometry>
+            </collision>
 			<visual>
 				<origin rpy="0 0 0" xyz="0 0 0" />
@@ -112,4 +123,10 @@
 				<inertia ixx="0.177" ixy="-2.34e-06" ixz="-4.92e-06" iyy="0.161" iyz="-0.05" izz="0.022" />
 			</inertial>
+            <collision>
+                <origin rpy="-0.55 0 0" xyz="0 0.075 -0.16" />
+                <geometry>
+                    <cylinder radius="0.05" length="0.4"/>
+                </geometry>
+            </collision>
 			<visual>
 				<origin rpy="0 0 0" xyz="0 0 0" />
@@ -140,4 +157,10 @@
 				<inertia ixx="0.007" ixy="-4.93e-06" ixz="-5.57e-06" iyy="0.004" iyz="-6.64e-05" izz="0.007" />
 			</inertial>
+            <collision>
+                <origin rpy="1.571 0 0" xyz="0 0 0" />
+                <geometry>
+                    <cylinder radius="0.06" length="0.15"/>
+                </geometry>
+            </collision>
 			<visual>
 				<origin rpy="0 0 0" xyz="0 0 0" />

File: dsr_description/xacro/macro.m1509.white.xacro (robot description, xacro)
@@ -34,4 +34,9 @@
 				<inertia ixx="0.039" ixy="2.1e-05" ixz="-3.61e-05" iyy="0.023" iyz="-0.003" izz="0.039" />
 			</inertial>
+            <collision>
+                <geometry>
+                    <cylinder radius="0.08" length="0.2"/>
+                </geometry>
+            </collision>
 			<visual>
 				<origin rpy="0 0 0" xyz="0 0 0" />
@@ -56,4 +61,10 @@
 				<inertia ixx="0.820" ixy="1.19e-05" ixz="-0.000263" iyy="0.82" iyz="-0.008" izz="0.031" />
 			</inertial>
+            <collision>
+                <origin rpy="0 -1.571 0" xyz="0.2 0 0.1525" />
+                <geometry>
+                    <cylinder radius="0.08" length="0.5"/>
+                </geometry>
+            </collision>
 			<visual>
 				<origin rpy="0 0 0" xyz="0 0 0" />
@@ -112,4 +123,10 @@
 				<inertia ixx="0.177" ixy="-2.34e-06" ixz="-4.92e-06" iyy="0.161" iyz="-0.05" izz="0.022" />
 			</inertial>
+            <collision>
+                <origin rpy="-0.55 0 0" xyz="0 0.075 -0.16" />
+                <geometry>
+                    <cylinder radius="0.05" length="0.4"/>
+                </geometry>
+            </collision>
 			<visual>
 				<origin rpy="0 0 0" xyz="0 0 0" />
@@ -140,4 +157,10 @@
 				<inertia ixx="0.007" ixy="-4.93e-06" ixz="-5.57e-06" iyy="0.004" iyz="-6.64e-05" izz="0.007" />
 			</inertial>
+            <collision>
+                <origin rpy="1.571 0 0" xyz="0 0 0" />
+                <geometry>
+                    <cylinder radius="0.06" length="0.15"/>
+                </geometry>
+            </collision>
 			<visual>
 				<origin rpy="0 0 0" xyz="0 0 0" />
